File: inputs.kicad_sch (KiCad schematic)
At the start: 110 parts, among them J10 Screw_Terminal_01x06, J14 Screw_Terminal_01x04, J16 Screw_Terminal_01x06, J18 Screw_Terminal_01x06, J19 Screw_Terminal_01x06, J9 Screw_Terminal_01x06, U7 MC33978

Commit message: routed inputs and outputs
Connections:
- net _SP8 is gone; now on net _SG8: R51.2, U7.19 (SG8)
- net _SG6: now also R31.2, U7.15 (SG6)
- net WAKE_B0: no longer names the net of R28.2, U7.17 (WAKE_B)
Other:
- moved on the sheet: C33, C34, C35, C36, C37, C38, C39, C40, C41, C42, C43
