File: outputs2.kicad_sch (KiCad schematic)
At the start: 82 parts, among them J3 Screw_Terminal_01x06, J5 Screw_Terminal_01x06, J6 Screw_Terminal_01x06, U1 DRV8876, U10 BTS7008, U11 BTS7008, U14 DRV8876, U8 BTS7008, U9 BTS7008

Commit message: routed inputs and outputs
Parts:
- renumbered C62 to C61, C61 to C62
Connections:
- net nSLEEPn renamed nSLEEPMn
Other:
- moved on the sheet: C49, C51, R54, R55, R57
