File: processor.kicad_sch (KiCad schematic)
At the start: 38 parts, among them J1 AVR-ISP-6, J4 Screw_Terminal_01x04, Q3 2N7002, Q4 2N7002, SW2 EVQ-P9W02W, U2 ATmega1284P-A, U3 MCP2515, U6 MCP2562-E-MF, Y1 16MHz, Y2 12MHz

Commit message: routed inputs and outputs
Parts:
- added C71, C72, C73: .1uF, Capacitor_SMD:C_0603_1608Metric, symbol Device:C_Polarized_Small_US
Connections:
- net +3.3V: now also C72.1, C73.1
- net GND: now also C71.2, C72.2, C73.2
- net at C10.1, L3.2, U2.27 (AVCC): now also C71.1
- net ADC2 renamed IPROPIM0
- net ADC3 renamed IPROPIM1
Other:
- moved on the sheet: C10, C9, L3

Commit message: mostly routed
Connections:
- net ADC1: no longer names the net of C16.1, D1.2, R27.1, U2.36 (PA1)
Changed lines of the file:
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@@
 	(wire
 		(pts
-			(xy 100.33 120.65) (xy 109.22 120.65)
+			(xy 100.33 120.65) (xy 110.49 120.65)
 		)
 		(stroke
@@
 	(wire
 		(pts
-			(xy 100.33 125.73) (xy 109.22 125.73)
+			(xy 100.33 125.73) (xy 110.49 125.73)
 		)
 		(stroke
@@
 	(wire
 		(pts
-			(xy 100.33 158.75) (xy 114.3 158.75)
-		)
-		(stroke
-			(width 0)
-			(type default)
-		)
-	)
-	(wire
-		(pts
 			(xy 194.31 128.27) (xy 194.31 130.81)
 		)
@@
 	(wire
 		(pts
+			(xy 100.33 158.75) (xy 106.68 158.75)
+		)
+		(stroke
+			(width 0)
+			(type default)
+		)
+	)
+	(wire
+		(pts
 			(xy 25.4 95.25) (xy 25.4 93.98)
 		)
@@
 	(wire
 		(pts
-			(xy 100.33 123.19) (xy 109.22 123.19)
+			(xy 100.33 123.19) (xy 110.49 123.19)
 		)
 		(stroke
@@
 		)
 	)
-	(label "ADC1"
-		(at 102.87 87.63 0)
-		(effects
-			(font
-				(size 1.27 1.27)
-			)
-			(justify left bottom)
-		)
-	)
-	(label "SCLK0"
-		(at 102.87 125.73 0)
-		(effects
-			(font
-				(size 1.27 1.27)
-			)
-			(justify left bottom)
-		)
-	)
 	(label "RST"
 		(at 67.31 85.09 180)
@@
 	)
 	(label "INT_CAN0"
-		(at 114.3 158.75 0)
+		(at 102.87 158.75 0)
 		(effects
 			(font
@@
 		)
 	)
-	(label "AMUX0"
-		(at 102.87 85.09 0)
-		(effects
-			(font
-				(size 1.27 1.27)
-			)
-			(justify left bottom)
-		)
-	)
 	(label "CS_CAN"
 		(at 102.87 107.95 0)
@@
 		)
 	)
-	(label "INT_B0"
-		(at 102.87 113.03 0)
-		(effects
-			(font
-				(size 1.27 1.27)
-			)
-			(justify left bottom)
-		)
-	)
-	(label "MOSI0"
-		(at 102.87 120.65 0)
-		(effects
-			(font
-				(size 1.27 1.27)
-			)
-			(justify left bottom)
-		)
-	)
 	(label "MISO0"
 		(at 179.07 43.18 0)
@@
 		)
 	)
-	(label "CS_IN0"
-		(at 102.87 110.49 0)
-		(effects
-			(font
-				(size 1.27 1.27)
-			)
-			(justify left bottom)
-		)
-	)
 	(label "RX0"
 		(at 102.87 153.67 0)
@@
 		)
 	)
-	(label "MISO0"
-		(at 102.87 123.19 0)
-		(effects
-			(font
-				(size 1.27 1.27)
-			)
-			(justify left bottom)
-		)
-	)
 	(label "MOSI0"
 		(at 179.07 40.64 0)
@@
 		)
 	)
-	(label "ADC3"
-		(at 102.87 92.71 0)
-		(effects
-			(font
-				(size 1.27 1.27)
-			)
-			(justify left bottom)
-		)
-	)
 	(label "SCLK0"
 		(at 179.07 48.26 0)
@@
 	(label "INT_CAN0"
 		(at 224.79 55.88 0)
-		(effects
-			(font
-				(size 1.27 1.27)
-			)
-			(justify left bottom)
-		)
-	)
-	(label "ADC2"
-		(at 102.87 90.17 0)
 		(effects
 			(font
@@
 			(hide yes)
 			(show_name no)
-			(do_not_autoplace no)
-			(effects
-				(font
-					(size 1.27 1.27)
-				)
-				(justify left)
-			)
-		)
-	)
-	(global_label "WAKE_B0"
-		(shape input)
-		(at 167.64 114.3 0)
-		(fields_autoplaced yes)
-		(effects
-			(font
-				(size 1.27 1.27)
-			)
-			(justify left)
-		)
-		(property "Intersheetrefs" "${INTERSHEET_REFS}"
-			(at 179.0313 114.3 0)
-			(hide yes)
-			(show_name no)
