File: robust-io.kicad_pcb (KiCad board)
At the start: 4 copper layers, 255 parts, among them J1 AVR-ISP-6, J10 Screw_Terminal_01x06, J14 Screw_Terminal_01x04, J15 Screw_Terminal_01x04, J16 Screw_Terminal_01x06, J18 Screw_Terminal_01x06, J19 Screw_Terminal_01x06, J3 Screw_Terminal_01x06, J4 Screw_Terminal_01x04, J5 Screw_Terminal_01x06, J6 Screw_Terminal_01x06, J9 Screw_Terminal_01x06, Q3 2N7002, Q4 2N7002, SW2 EVQ-P9W02W, U1 DRV8876, U10 BTS7008, U11 BTS7008, U14 DRV8876, U2 ATmega1284P-A, U3 MCP2515, U4 TPS5604, U5 TPS5604, U6 MCP2562-E-MF, U7 MC33978, U8 BTS7008, U9 BTS7008, Y1 16MHz, Y2 12MHz

Commit message: routed inputs and outputs
Parts:
- added C71: .1uF, Capacitor_SMD:C_0603_1608Metric, F.Cu at (153.6, 80.2)
- added C72: .1uF, Capacitor_SMD:C_0603_1608Metric, F.Cu at (143.2, 69.1)
- added C73: .1uF, Capacitor_SMD:C_0603_1608Metric, F.Cu at (151.6, 84.9)
- moved R25 51.2 mm to (109.3, 98.7), turned to -90 degrees
- moved R26 49.3 mm to (111.1, 98.7), turned to -90 degrees
- moved D5 47.3 mm to (110.2, 95.3), turned to 180 degrees
- moved R88 37.1 mm to (152.4, 154.9)
- moved R89 37.1 mm to (156.5, 154.9)
- moved R90 37.1 mm to (160.5, 154.9)
- moved R91 37.1 mm to (164.6, 154.9)
- moved D40 37.1 mm to (151.5, 157.2)
- moved D41 37.1 mm to (155.5, 157.2)
- moved D42 37.1 mm to (159.6, 157.2)
- moved D43 37.1 mm to (163.7, 157.2)
- moved R55 31.6 mm to (164.6, 107.3)
- moved R54 31.6 mm to (168.7, 108.2)
- moved C51 31.5 mm to (168.7, 106.5)
- moved R57 19.3 mm to (149.9, 117.3), turned to -90 degrees
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- renumbered C62 to C61, C61 to C62
Connections:
- net /inputs/WAKE_B0 renamed Net-(U7-WAKE_B)
- net /outputs2/ISENSE renamed ISENSE
- C21 pad 1: /inputs/AMUX0 -> AMUX0
- C48 pad 1: /outputs2/IPROPIM1 -> IPROPIM1
- C49 pad 1: /outputs2/IPROPIM0 -> IPROPIM0
- D1 pad 1: /processor/AMUX0 -> AMUX0
- D3 pad 1: /processor/ADC3 -> IPROPIM1
- D3 pad 2: /processor/ADC2 -> IPROPIM0
- D5 pad 1: /outputs2/ISENSE_PROT -> ISENSE_PROT
- J1 pad 1: /processor/MISO0 -> MISO0
- J1 pad 3: /processor/SCLK0 -> SCLK0
- J1 pad 4: /processor/MOSI0 -> MOSI0
- R10 pad 1: /outputs2/DEN0 -> DEN0
- R11 pad 1: /outputs2/DSELn -> DSELn
- R12 pad 1: /outputs2/DRV_OUT1 -> DRV_OUT1
- R13 pad 1: /outputs2/DRV_OUT2 -> DRV_OUT2
- R14 pad 1: /outputs2/DEN1 -> DEN1
- R15 pad 1: /outputs2/DSELn -> DSELn
- R16 pad 1: /outputs2/DRV_OUT3 -> DRV_OUT3
- R17 pad 1: /outputs2/DRV_OUT4 -> DRV_OUT4
- R18 pad 1: /outputs2/DEN2 -> DEN2
- R19 pad 1: /outputs2/DSELn -> DSELn
- R20 pad 1: /outputs2/DRV_OUT5 -> DRV_OUT5
- R21 pad 1: /outputs2/DRV_OUT6 -> DRV_OUT6
- R22 pad 1: /outputs2/DEN3 -> DEN3
- R23 pad 1: /outputs2/DSELn -> DSELn
- R24 pad 1: /outputs2/DRV_OUT7 -> DRV_OUT7
- R26 pad 1: /outputs2/ISENSE_PROT -> ISENSE_PROT
- R27 pad 2: /processor/ISENSE_PROT -> ISENSE_PROT
- R29 pad 1: /inputs/INT_B0 -> INT_B0
- R30 pad 1: /inputs/AMUX0 -> AMUX0
- R31 pad 2: Net-(U7-SG6) -> /inputs/_SG6
- R51 pad 2: /inputs/_SP8 -> /inputs/_SG8
- R53 pad 2: /outputs2/FAULTMn -> FAULTMn
- R56 pad 1: /outputs2/IPROPIM1 -> IPROPIM1
- R57 pad 1: /outputs2/IPROPIM0 -> IPROPIM0
- R9 pad 1: /outputs2/DRV_OUT0 -> DRV_OUT0
- U1 pad 1: /outputs2/EN_M1 -> EN_M1
- U1 pad 2: /outputs2/PH_M1 -> PH_M1
- U1 pad 3: /outputs2/nSLEEPn -> nSLEEPMn
- U1 pad 4: /outputs2/FAULTMn -> FAULTMn
- U1 pad 6: /outputs2/IPROPIM1 -> IPROPIM1
- U14 pad 1: /outputs2/EN_M0 -> EN_M0
- U14 pad 2: /outputs2/PH_M0 -> PH_M0
- U14 pad 3: /outputs2/nSLEEPn -> nSLEEPMn
- U14 pad 4: /outputs2/FAULTMn -> FAULTMn
- U14 pad 6: /outputs2/IPROPIM0 -> IPROPIM0
- U2 pad 1: /processor/MOSI0 -> MOSI0
- U2 pad 12: /processor/FAULTMn -> FAULTMn
- U2 pad 13: /processor/PH_M0 -> PH_M0
- U2 pad 14: /processor/EN_M0 -> EN_M0
- U2 pad 15: /processor/PH_M1 -> PH_M1
- U2 pad 16: /processor/EN_M1 -> EN_M1
- U2 pad 19: /processor/DRV_OUT0 -> DRV_OUT0
- U2 pad 2: /processor/MISO0 -> MISO0
- U2 pad 20: /processor/DRV_OUT1 -> DRV_OUT1
- U2 pad 21: /processor/DRV_OUT2 -> DRV_OUT2
- U2 pad 22: /processor/DRV_OUT3 -> DRV_OUT3
- U2 pad 23: /processor/DRV_OUT4 -> DRV_OUT4
- U2 pad 24: /processor/DRV_OUT5 -> DRV_OUT5
- U2 pad 25: /processor/DRV_OUT6 -> DRV_OUT6
- U2 pad 26: /processor/DRV_OUT7 -> DRV_OUT7
- U2 pad 3: /processor/SCLK0 -> SCLK0
- U2 pad 30: /processor/nSLEEPMn -> nSLEEPMn
- U2 pad 31: /processor/DSELn -> DSELn
- U2 pad 32: /processor/DEN3 -> DEN3
- U2 pad 33: /processor/DEN2 -> DEN2
- U2 pad 34: /processor/ADC3 -> IPROPIM1
- U2 pad 35: /processor/ADC2 -> IPROPIM0
- U2 pad 37: /processor/AMUX0 -> AMUX0
- U2 pad 41: /processor/CS_IN0 -> CS_IN0
- U2 pad 42: /processor/INT_B0 -> INT_B0
- U2 pad 43: /processor/DEN0 -> DEN0
- U2 pad 44: /processor/DEN1 -> DEN1
- U3 pad 13: /processor/SCLK0 -> SCLK0
- U3 pad 14: /processor/MOSI0 -> MOSI0
- U3 pad 15: /processor/MISO0 -> MISO0
- U7 pad 15: Net-(U7-SG6) -> /inputs/_SG6
- U7 pad 19: /inputs/_SP8 -> /inputs/_SG8
- U7 pad 2: /inputs/MOSI0 -> MOSI0
- U7 pad 29: /inputs/INT_B0 -> INT_B0
- U7 pad 3: /inputs/SCLK0 -> SCLK0
- U7 pad 32: /inputs/MISO0 -> MISO0
- U7 pad 4: /inputs/CS_IN0 -> CS_IN0
Routing:
- net /inputs/_SP4: track 0.00 -> 93.7 mm
- net /inputs/_SP5: track 0.00 -> 89.4 mm
- net GND: track 0.00 -> 89.3 mm, vias 0 -> 31
- net /inputs/_SP6: track 0.00 -> 85.4 mm
- net /inputs/_SP7: track 0.00 -> 81.5 mm
- net /inputs/_SG13: track 0.00 -> 78.1 mm
- net +24V: track 0.00 -> 74.5 mm, vias 0 -> 24
- net /inputs/_SG12: track 0.00 -> 73.9 mm
- net ISENSE: track 0.00 -> 70.2 mm, vias 0 -> 5
- net /inputs/_SG11: track 0.00 -> 60.3 mm
- net /inputs/_SP0: track 0.00 -> 56.8 mm
- net /inputs/_SG10: track 0.00 -> 56.7 mm
- net /inputs/_SP1: track 0.00 -> 53.2 mm
- net /inputs/_SG9: track 0.00 -> 52.3 mm
- net /inputs/_SP2: track 0.00 -> 49.9 mm
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- added copper zone on F.Cu, net /outputs2/OUT1M0
- added copper zone on F.Cu, net /outputs2/OUT_0
- added copper zone on F.Cu, net /outputs2/OUT_1
- added copper zone on F.Cu, net /outputs2/OUT_2
- added copper zone on F.Cu, net /outputs2/OUT_3
- added copper zone on F.Cu, net /outputs2/OUT_4
- added copper zone on F.Cu, net /outputs2/OUT_5
- added copper zone on F.Cu, net /outputs2/OUT_6
- added copper zone on F.Cu, net /outputs2/OUT_7
- added copper zone on In1.Cu, net GND
Other:
- board outline added: 159.1 x 101.4 mm

Commit message: mostly routed
Parts:
- C8: footprint Capacitor_SMD:C_0805_2012Metric_Pad1.18x1.45mm_HandSolder -> Capacitor_SMD:C_0603_1608Metric_Pad1.08x0.95mm_HandSolder
- moved R91 99.2 mm to (74.4, 113.7), turned to -90 degrees
- moved D43 98.0 mm to (74.4, 116.9)
- moved R90 97.3 mm to (72.4, 113.7), turned to -90 degrees
- moved D42 96.0 mm to (72.4, 117.0)
- moved R89 95.2 mm to (70.6, 113.7), turned to -90 degrees
- moved D41 94.0 mm to (70.6, 117.0)
- moved R88 93.3 mm to (68.7, 113.7), turned to -90 degrees
- moved D40 92.0 mm to (68.7, 116.9)
- moved R4 54.0 mm to (88.1, 83.9), turned to 180 degrees
- moved U4 48.4 mm to (84.8, 81.0), turned to 90 degrees
- moved R6 47.3 mm to (88.4, 72.2), turned to 180 degrees
- moved C3 46.0 mm to (84.7, 76.5), turned to 90 degrees
- moved C4 44.2 mm to (81.8, 81.1), turned to 90 degrees
- moved C6 43.3 mm to (85.0, 64.7), turned to 90 degrees
- moved U5 43.1 mm to (85.1, 69.3), turned to 90 degrees
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Connections:
- net /processor/ADC1 renamed Net-(U2-PA1)
Routing:
- net +3.3V: track 3.78 -> 152.3 mm, vias 0 -> 2
- net DSELn: track 0.00 -> 95.0 mm, vias 0 -> 5
- net GND: track 89.3 -> 164.6 mm, vias 31 -> 59
- net /outputs2/OUT_7: track 37.6 -> 106.8 mm, vias 0 -> 2
- net /outputs2/OUT_6: track 40.5 -> 102.0 mm, vias 0 -> 2
- net /outputs2/OUT_5: track 40.1 -> 95.4 mm, vias 0 -> 2
- net /processor/TX0: track 0.00 -> 49.2 mm, vias 0 -> 2
- net /outputs2/OUT_4: track 44.7 -> 93.7 mm, vias 0 -> 2
- net DEN0: track 0.00 -> 47.1 mm, vias 0 -> 2
- net /outputs2/OUT_3: track 42.6 -> 88.1 mm, vias 0 -> 2
- net /processor/RX0: track 0.00 -> 44.0 mm
- net /outputs2/OUT_2: track 40.9 -> 80.2 mm, vias 0 -> 2
- net DRV_OUT0: track 0.00 -> 38.2 mm
- net DEN3: track 0.00 -> 36.2 mm, vias 0 -> 2
- net DRV_OUT7: track 0.00 -> 34.1 mm
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