File: _claude_scratch/outputs2.before-erc.kicad_sch (KiCad schematic)
At the start: 82 parts, among them J3 Screw_Terminal_01x06, J5 Screw_Terminal_01x06, J6 Screw_Terminal_01x06, U1 DRV8876, U10 BTS7008, U11 BTS7008, U14 DRV8876, U8 BTS7008, U9 BTS7008

Commit message: Rev A: release to fab (JLCPCB, 5 PCB / 2 assembled)
Board
- Outline set to exactly 160 x 100 mm; plane zones resized to match
- UART brought out on J20 (1x6 SMD, FTDI pinout) with series
  resistors R98/R99 and TVS D48
- J1 and J20 changed to SMD headers (C52016780, C41417363)
- L1/L2 moved to Sunlord SWPA4030S footprints; regulator tracks rerouted
- 41 test points added (35 top, 6 bottom), including SPI access
- Crystal case pins (Y1/Y2 pads 2, 4) tied to GND
- SW2 changed to 2-pin push button symbol
- R84-R91 changed from 2.2k to 10k to cut dissipation at 24 V
- Thermal vias in U1/U14 enlarged to 0.3 mm drill; 27 +24V vias added
  under U8-U11; solid plane connections on high-current pins
- Input/output rows and edge connectors aligned
- /inputs/_SG4 track and via moved clear of R74 pad 1

Schematic
- ERC cleared: no-connects, PWR_FLAGs, pin types, off-grid items
- Symbols moved to project library robust-io
- Test point symbols added on processor and power sheets

Rules
- Custom DRC rule for U7 pad-to-pad clearance (0.15 mm)
- Minimum through hole 0.2 mm; silk-to-edge check ignored

Fab outputs (fab/)
- make_gerbers.sh: Gerbers, drill and position export via kicad-cli
- JLC BOM with LCSC part numbers on all 50 SMD lines
- JLC placement file with per-part rotation offsets
  (cpl_rotation_offsets.json), verified in JLC placement preview
- Through-hole BOM and test point list

DRC: 4 library-mismatch warnings (J20, U1, U14, U7), 0 errors
ERC: clean
Parts:
- R84, R85, R86, R87, R88, R89, R90, R91: value 10k -> 2.2k
- U1, U14: symbol robust-io:DRV8876PWPR -> rml_kicad_lib:DRV8876PWPR
- U10, U11, U8, U9: symbol robust-io:BTS7008-2EPA -> rml_kicad_lib:BTS7008-2EPA
Changed lines of the file:
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@@
 	(wire
 		(pts
-			(xy 261.62 64.77) (xy 271.78 64.77)
+			(xy 250.19 64.77) (xy 271.78 64.77)
 		)
 		(stroke
@@
 	(wire
 		(pts
-			(xy 271.78 41.91) (xy 261.62 41.91)
+			(xy 271.78 41.91) (xy 250.19 41.91)
 		)
 		(stroke
@@
 	(wire
 		(pts
-			(xy 252.73 85.09) (xy 271.78 85.09)
+			(xy 250.19 85.09) (xy 271.78 85.09)
 		)
 		(stroke
@@
 	(wire
 		(pts
-			(xy 261.62 59.69) (xy 271.78 59.69)
+			(xy 250.19 59.69) (xy 271.78 59.69)
 		)
 		(stroke
@@
 	(wire
 		(pts
-			(xy 271.78 46.99) (xy 261.62 46.99)
+			(xy 271.78 46.99) (xy 250.19 46.99)
 		)
 		(stroke
@@
 	(wire
 		(pts
-			(xy 252.73 77.47) (xy 271.78 77.47)
+			(xy 250.19 77.47) (xy 271.78 77.47)
 		)
 		(stroke
@@
 	(wire
 		(pts
-			(xy 252.73 80.01) (xy 271.78 80.01)
+			(xy 250.19 80.01) (xy 271.78 80.01)
 		)
 		(stroke
@@
 	(wire
 		(pts
-			(xy 261.62 62.23) (xy 271.78 62.23)
+			(xy 250.19 62.23) (xy 271.78 62.23)
 		)
 		(stroke
@@
 	(wire
 		(pts
-			(xy 271.78 49.53) (xy 261.62 49.53)
+			(xy 271.78 49.53) (xy 250.19 49.53)
 		)
 		(stroke
@@
 	(wire
 		(pts
-			(xy 252.73 82.55) (xy 271.78 82.55)
+			(xy 250.19 82.55) (xy 271.78 82.55)
 		)
 		(stroke
@@
 	(wire
 		(pts
-			(xy 271.78 44.45) (xy 261.62 44.45)
+			(xy 271.78 44.45) (xy 250.19 44.45)
 		)
 		(stroke
@@
 	(wire
 		(pts
-			(xy 261.62 67.31) (xy 271.78 67.31)
+			(xy 250.19 67.31) (xy 271.78 67.31)
 		)
 		(stroke
@@
 	)
 	(symbol
-		(lib_id "robust-io:DRV8876PWPR")
+		(lib_id "rml_kicad_lib:DRV8876PWPR")
 		(at 186.69 59.69 0)
 		(unit 1)
@@
 			)
 		)
-		(property "Value" "10k"
+		(property "Value" "2.2k"
 			(at 265.938 143.764 90)
 			(show_name no)
@@
 			)
 		)
-		(property "Value" "10k"
+		(property "Value" "2.2k"
 			(at 265.938 128.524 90)
 			(show_name no)
@@
 	)
 	(symbol
-		(lib_id "robust-io:BTS7008-2EPA")
+		(lib_id "rml_kicad_lib:BTS7008-2EPA")
 		(at 69.85 41.91 0)
 		(unit 1)
@@
 	)
 	(symbol
-		(lib_id "robust-io:BTS7008-2EPA")
+		(lib_id "rml_kicad_lib:BTS7008-2EPA")
 		(at 69.85 142.24 0)
 		(unit 1)
@@
 	)
 	(symbol
-		(lib_id "robust-io:DRV8876PWPR")
+		(lib_id "rml_kicad_lib:DRV8876PWPR")
 		(at 186.69 105.41 0)
 		(unit 1)
@@
 	)
 	(symbol
-		(lib_id "robust-io:BTS7008-2EPA")
+		(lib_id "rml_kicad_lib:BTS7008-2EPA")
 		(at 69.85 74.93 0)
 		(unit 1)
@@
 			)
 		)
-		(property "Value" "10k"
+		(property "Value" "2.2k"
 			(at 265.938 113.284 90)
 			(show_name no)
@@
 	)
 	(symbol
-		(lib_id "robust-io:BTS7008-2EPA")
+		(lib_id "rml_kicad_lib:BTS7008-2EPA")
 		(at 69.85 107.95 0)
 		(unit 1)
@@
 			)
 		)
-		(property "Value" "10k"
+		(property "Value" "2.2k"
 			(at 265.938 148.844 90)
 			(show_name no)
@@
 			)
 		)
-		(property "Value" "10k"
+		(property "Value" "2.2k"
 			(at 265.938 138.684 90)
 			(show_name no)
@@
 			)
 		)
-		(property "Value" "10k"
+		(property "Value" "2.2k"
 			(at 265.938 123.444 90)
 			(show_name no)
@@
 			)
 		)
-		(property "Value" "10k"
+		(property "Value" "2.2k"
 			(at 265.938 133.604 90)
 			(show_name no)
@@
 			)
 		)
-		(property "Value" "10k"
+		(property "Value" "2.2k"
 			(at 265.938 118.364 90)
 			(show_name no)
