File: _claude_scratch/processor.before-sw2.kicad_sch (KiCad schematic)
At the start: 51 parts, among them J1 AVR-ISP-6, J20 UART 3V3 (FTDI pinout), J4 Screw_Terminal_01x04, Q3 2N7002, Q4 2N7002, SW1 CHS-01TB, SW2 B3U-1000P, U2 ATmega1284P-A, U3 MCP2515, U6 MCP2562-E-MF, Y1 16MHz, Y2 12MHz

Commit message: Rev A: release to fab (JLCPCB, 5 PCB / 2 assembled)
Board
- Outline set to exactly 160 x 100 mm; plane zones resized to match
- UART brought out on J20 (1x6 SMD, FTDI pinout) with series
  resistors R98/R99 and TVS D48
- J1 and J20 changed to SMD headers (C52016780, C41417363)
- L1/L2 moved to Sunlord SWPA4030S footprints; regulator tracks rerouted
- 41 test points added (35 top, 6 bottom), including SPI access
- Crystal case pins (Y1/Y2 pads 2, 4) tied to GND
- SW2 changed to 2-pin push button symbol
- R84-R91 changed from 2.2k to 10k to cut dissipation at 24 V
- Thermal vias in U1/U14 enlarged to 0.3 mm drill; 27 +24V vias added
  under U8-U11; solid plane connections on high-current pins
- Input/output rows and edge connectors aligned
- /inputs/_SG4 track and via moved clear of R74 pad 1

Schematic
- ERC cleared: no-connects, PWR_FLAGs, pin types, off-grid items
- Symbols moved to project library robust-io
- Test point symbols added on processor and power sheets

Rules
- Custom DRC rule for U7 pad-to-pad clearance (0.15 mm)
- Minimum through hole 0.2 mm; silk-to-edge check ignored

Fab outputs (fab/)
- make_gerbers.sh: Gerbers, drill and position export via kicad-cli
- JLC BOM with LCSC part numbers on all 50 SMD lines
- JLC placement file with per-part rotation offsets
  (cpl_rotation_offsets.json), verified in JLC placement preview
- Through-hole BOM and test point list

DRC: 4 library-mismatch warnings (J20, U1, U14, U7), 0 errors
ERC: clean
Parts:
- removed D48: SP0502BAHT, Package_TO_SOT_SMD:SOT-23, symbol Power_Protection:SP0502BAHT
- removed J20: UART 3V3 (FTDI pinout), Connector_PinHeader_2.54mm:PinHeader_1x06_P2.54mm_Vertical_SMD_Pin1Right, symbol Connector_Generic:Conn_01x06
- removed R98, R99: 1k, Resistor_SMD:R_0603_1608Metric, symbol Device:R_US
- removed SW1: CHS-01TB, Button_Switch_SMD:SW_DIP_SPSTx01_Slide_Copal_CHS-01B_W7.62mm_P1.27mm, symbol Switch:SW_DIP_x01
- removed TP10: INT_CAN0, TestPoint:TestPoint_Pad_D1.0mm, symbol Connector:TestPoint
- removed TP11: RST, TestPoint:TestPoint_Pad_D1.0mm, symbol Connector:TestPoint
- removed TP12: RX0, TestPoint:TestPoint_Pad_D1.0mm, symbol Connector:TestPoint
- removed TP13: TX0, TestPoint:TestPoint_Pad_D1.0mm, symbol Connector:TestPoint
- removed TP8: CS_CAN, TestPoint:TestPoint_Pad_D1.0mm, symbol Connector:TestPoint
- SW2: value B3U-1000P -> EVQ-P9W02W; footprint Button_Switch_SMD:SW_SPST_B3U-1000P -> rml:KEY-SMD_EVQP9W02W; symbol Switch:SW_Push -> rml_kicad_lib:SW_SPST_PB
- U2: symbol robust-io:ATmega1284P-A -> MCU_Microchip_ATmega:ATmega1284P-A
- U3: symbol robust-io:MCP2515-xSO -> Interface_CAN_LIN:MCP2515-xSO
- U6: symbol robust-io:MCP2562-E-MF -> Interface_CAN_LIN:MCP2562-E-MF
- Y1, Y2: symbol robust-io:Crystal_4Pin_3.2x2.5mm -> rml_kicad_lib:Crystal_4Pin_3.2x2.5mm
Connections:
- net GND: no longer Y1.2, Y1.4, Y2.2, Y2.4
- net RST: now also SW2.2 (A), SW2.3 (C)
- net at R8.2: now also SW2.3 (C), SW2.4 (B); no longer SW2.2
- net at R2.1: now also J4.1 (Pin_1), U6.7 (CANH)
- no-connect marks 8 -> 0
Other:
- moved on the sheet: C69, C70, D44, D45, D46, D47, Q3, Q4, R92, R93, R95, R97
